Commit message: Increase robot weight per SpaceEngineer's block weight
https://spaceengineers-archive.fandom.com/wiki/Light_Armor_Block

It weights 20kg and its side lenght is 0.5m

File: resources/robots/v0/urdf/v0.urdf.xacro (robot description, xacro)
@@ -16,9 +16,10 @@
         </collision>
 		<inertial>
-			<mass value="${sizeX * sizeY * sizeZ * 50.}" />
+			<xacro:property name="weight" value="${sizeX * sizeY * sizeZ * 160}"/>
+			<mass value="${weight}"/>
 			<inertia
-				ixx="${1.0/12.0 * sizeX * sizeY * sizeZ * 50 * (sizeZ * sizeZ + sizeY * sizeY)}"
-				iyy="${1.0/12.0 * sizeX * sizeY * sizeZ * 50 * (sizeZ * sizeZ + sizeX * sizeX)}"
-				izz="${1.0/12.0 * sizeX * sizeY * sizeZ * 50 * (sizeY * sizeY + sizeX * sizeX)}"
+				ixx="${1.0/12.0 * weight * (sizeZ * sizeZ + sizeY * sizeY)}"
+				iyy="${1.0/12.0 * weight * (sizeZ * sizeZ + sizeX * sizeX)}"
+				izz="${1.0/12.0 * weight * (sizeY * sizeY + sizeX * sizeX)}"
 				ixy="0.0" ixz="0.0" iyz="0.0"/>
 		</inertial>

File: resources/robots/v0/urdf/v0_weight_50.urdf (robot description, URDF)
Before this commit: robot v0, 17 links, 16 joints
Links:
- link body: mass 6.240000000000001 -> 1.9500000000000004
- link l1_segment_1: mass 0.32000000000000006 -> 0.10000000000000002
- link l1_segment_2_HIP: mass 0.96 -> 0.3
- link l1_segment_3_THIGH: mass 1.12 -> 0.35000000000000003
- link l1_segment_4_FOOT: mass 0.6400000000000001 -> 0.20000000000000004
- link l3_segment_1: mass 0.32000000000000006 -> 0.10000000000000002
- link l3_segment_2_HIP: mass 0.96 -> 0.3
- link l3_segment_3_THIGH: mass 1.12 -> 0.35000000000000003
- link l3_segment_4_FOOT: mass 0.6400000000000001 -> 0.20000000000000004
- link r1_segment_1: mass 0.32000000000000006 -> 0.10000000000000002
- link r1_segment_2_HIP: mass 0.96 -> 0.3
- link r1_segment_3_THIGH: mass 1.12 -> 0.35000000000000003
- link r1_segment_4_FOOT: mass 0.6400000000000001 -> 0.20000000000000004
- link r3_segment_1: mass 0.32000000000000006 -> 0.10000000000000002
- link r3_segment_2_HIP: mass 0.96 -> 0.3
- link r3_segment_3_THIGH: mass 1.12 -> 0.35000000000000003
- link r3_segment_4_FOOT: mass 0.6400000000000001 -> 0.20000000000000004

File: resources/robots/v0six/urdf/v0.urdf (robot description, URDF)
Before this commit: robot v0, 25 links, 24 joints
Links:
- link body: mass 1.9500000000000004 -> 6.240000000000001
- link l1_segment_1: mass 0.10000000000000002 -> 0.32000000000000006
- link l1_segment_2_HIP: mass 0.3 -> 0.96
- link l1_segment_3_THIGH: mass 0.35000000000000003 -> 1.12
- link l1_segment_4_FOOT: mass 0.20000000000000004 -> 0.6400000000000001
- link l2_segment_1: mass 0.10000000000000002 -> 0.32000000000000006
- link l2_segment_2_HIP: mass 0.3 -> 0.96
- link l2_segment_3_THIGH: mass 0.35000000000000003 -> 1.12
- link l2_segment_4_FOOT: mass 0.20000000000000004 -> 0.6400000000000001
- link l3_segment_1: mass 0.10000000000000002 -> 0.32000000000000006
- link l3_segment_2_HIP: mass 0.3 -> 0.96
- link l3_segment_3_THIGH: mass 0.35000000000000003 -> 1.12
- link l3_segment_4_FOOT: mass 0.20000000000000004 -> 0.6400000000000001
- link r1_segment_1: mass 0.10000000000000002 -> 0.32000000000000006
- link r1_segment_2_HIP: mass 0.3 -> 0.96
- link r1_segment_3_THIGH: mass 0.35000000000000003 -> 1.12
- link r1_segment_4_FOOT: mass 0.20000000000000004 -> 0.6400000000000001
- link r2_segment_1: mass 0.10000000000000002 -> 0.32000000000000006
- link r2_segment_2_HIP: mass 0.3 -> 0.96
- link r2_segment_3_THIGH: mass 0.35000000000000003 -> 1.12
- link r2_segment_4_FOOT: mass 0.20000000000000004 -> 0.6400000000000001
- link r3_segment_1: mass 0.10000000000000002 -> 0.32000000000000006
- link r3_segment_2_HIP: mass 0.3 -> 0.96
- link r3_segment_3_THIGH: mass 0.35000000000000003 -> 1.12
- link r3_segment_4_FOOT: mass 0.20000000000000004 -> 0.6400000000000001
Joints:
- joint l1_joint_1_to_2: limit lower=-1.2 upper=1.2 effort=10 velocity=200 -> lower=-1.2 upper=1.2 effort=55 velocity=29
- joint l1_joint_2_to_3: limit lower=-0.2 upper=0.75 effort=10 velocity=90 -> lower=-0.2 upper=0.75 effort=55 velocity=29
- joint l1_joint_3_to_4_FOOT: limit lower=-0.2 upper=0.5 effort=10 velocity=70 -> lower=-0.2 upper=0.5 effort=55 velocity=29
- joint l2_joint_1_to_2: limit lower=-1.2 upper=1.2 effort=10 velocity=200 -> lower=-1.2 upper=1.2 effort=55 velocity=29
- joint l2_joint_2_to_3: limit lower=-0.2 upper=0.75 effort=10 velocity=90 -> lower=-0.2 upper=0.75 effort=55 velocity=29
- joint l2_joint_3_to_4_FOOT: limit lower=-0.2 upper=0.5 effort=10 velocity=70 -> lower=-0.2 upper=0.5 effort=55 velocity=29
- joint l3_joint_1_to_2: limit lower=-1.2 upper=1.2 effort=10 velocity=200 -> lower=-1.2 upper=1.2 effort=55 velocity=29
- joint l3_joint_2_to_3: limit lower=-0.2 upper=0.75 effort=10 velocity=90 -> lower=-0.2 upper=0.75 effort=55 velocity=29
- joint l3_joint_3_to_4_FOOT: limit lower=-0.2 upper=0.5 effort=10 velocity=70 -> lower=-0.2 upper=0.5 effort=55 velocity=29
- joint r1_joint_1_to_2: limit lower=-1.2 upper=1.2 effort=10 velocity=200 -> lower=-1.2 upper=1.2 effort=55 velocity=29
- joint r1_joint_2_to_3: limit lower=-0.75 upper=0.2 effort=10 velocity=90 -> lower=-0.75 upper=0.2 effort=55 velocity=29
- joint r1_joint_3_to_4_FOOT: limit lower=-0.5 upper=0.2 effort=10 velocity=70 -> lower=-0.5 upper=0.2 effort=55 velocity=29
- joint r2_joint_1_to_2: limit lower=-1.2 upper=1.2 effort=10 velocity=200 -> lower=-1.2 upper=1.2 effort=55 velocity=29
- joint r2_joint_2_to_3: limit lower=-0.75 upper=0.2 effort=10 velocity=90 -> lower=-0.75 upper=0.2 effort=55 velocity=29
- joint r2_joint_3_to_4_FOOT: limit lower=-0.5 upper=0.2 effort=10 velocity=70 -> lower=-0.5 upper=0.2 effort=55 velocity=29
- joint r3_joint_1_to_2: limit lower=-1.2 upper=1.2 effort=10 velocity=200 -> lower=-1.2 upper=1.2 effort=55 velocity=29
- joint r3_joint_2_to_3: limit lower=-0.75 upper=0.2 effort=10 velocity=90 -> lower=-0.75 upper=0.2 effort=55 velocity=29
- joint r3_joint_3_to_4_FOOT: limit lower=-0.5 upper=0.2 effort=10 velocity=70 -> lower=-0.5 upper=0.2 effort=55 velocity=29

File: resources/robots/v0six/urdf/v0.urdf.xacro (robot description, xacro)
@@ -16,9 +16,10 @@
         </collision>
 		<inertial>
-			<mass value="${sizeX * sizeY * sizeZ * 50.}" />
+			<xacro:property name="weight" value="${sizeX * sizeY * sizeZ * 160}"/>
+			<mass value="${weight}"/>
 			<inertia
-				ixx="${1.0/12.0 * sizeX * sizeY * sizeZ * 50 * (sizeZ * sizeZ + sizeY * sizeY)}"
-				iyy="${1.0/12.0 * sizeX * sizeY * sizeZ * 50 * (sizeZ * sizeZ + sizeX * sizeX)}"
-				izz="${1.0/12.0 * sizeX * sizeY * sizeZ * 50 * (sizeY * sizeY + sizeX * sizeX)}"
+				ixx="${1.0/12.0 * weight * (sizeZ * sizeZ + sizeY * sizeY)}"
+				iyy="${1.0/12.0 * weight * (sizeZ * sizeZ + sizeX * sizeX)}"
+				izz="${1.0/12.0 * weight * (sizeY * sizeY + sizeX * sizeX)}"
 				ixy="0.0" ixz="0.0" iyz="0.0"/>
 		</inertial>
@@ -45,5 +46,5 @@
 			<origin xyz="0 0 0.25" rpy="0 0 0" />
 			<axis xyz="0.0 0.0 1.0" />
-			<limit effort="10" lower="-1.2" upper="1.2" velocity="200"/>
+			<limit effort="55" lower="-1.2" upper="1.2" velocity="29"/>
 		</joint>
 		<link name="${name}_segment_3_THIGH">
@@ -58,8 +59,8 @@
 			<axis xyz="1.0 0.0 0.0" />
 			<xacro:if value="${reflect == -1}">
-				<limit effort="10" lower="-0.75" upper="0.2" velocity="90"/>
+				<limit effort="55" lower="-0.75" upper="0.2" velocity="29"/>
 			</xacro:if>
 			<xacro:unless value="${reflect == -1}">
-				<limit effort="10" lower="-0.2" upper="0.75" velocity="90"/>
+				<limit effort="55" lower="-0.2" upper="0.75" velocity="29"/>
 			</xacro:unless>
 		</joint>
@@ -75,8 +76,8 @@
 			<axis xyz="1.0 0.0 0.0" />
 			<xacro:if value="${reflect == -1}">
-				<limit effort="10" lower="-0.5" upper="0.2" velocity="70"/>
+				<limit effort="55" lower="-0.5" upper="0.2" velocity="29"/>
 			</xacro:if>
 			<xacro:unless value="${reflect == -1}">
-				<limit effort="10" lower="-0.2" upper="0.5" velocity="70"/>
+				<limit effort="55" lower="-0.2" upper="0.5" velocity="29"/>
 			</xacro:unless>
 		</joint>
