Commit message: v0: Adjust urdf joint limits
Increase effort and lower velocity

File: resources/robots/v0/urdf/v0.urdf (robot description, URDF)
Before this commit: robot v0, 17 links, 16 joints
Joints:
- joint l1_joint_1_to_2: limit lower=-1.2 upper=1.2 effort=10 velocity=200 -> lower=-1.2 upper=1.2 effort=55 velocity=29
- joint l1_joint_2_to_3: limit lower=-0.2 upper=0.75 effort=10 velocity=90 -> lower=-0.2 upper=0.75 effort=55 velocity=29
- joint l1_joint_3_to_4_FOOT: limit lower=-0.2 upper=0.5 effort=10 velocity=70 -> lower=-0.2 upper=0.5 effort=55 velocity=29
- joint l3_joint_1_to_2: limit lower=-1.2 upper=1.2 effort=10 velocity=200 -> lower=-1.2 upper=1.2 effort=55 velocity=29
- joint l3_joint_2_to_3: limit lower=-0.2 upper=0.75 effort=10 velocity=90 -> lower=-0.2 upper=0.75 effort=55 velocity=29
- joint l3_joint_3_to_4_FOOT: limit lower=-0.2 upper=0.5 effort=10 velocity=70 -> lower=-0.2 upper=0.5 effort=55 velocity=29
- joint r1_joint_1_to_2: limit lower=-1.2 upper=1.2 effort=10 velocity=200 -> lower=-1.2 upper=1.2 effort=55 velocity=29
- joint r1_joint_2_to_3: limit lower=-0.75 upper=0.2 effort=10 velocity=90 -> lower=-0.75 upper=0.2 effort=55 velocity=29
- joint r1_joint_3_to_4_FOOT: limit lower=-0.5 upper=0.2 effort=10 velocity=70 -> lower=-0.5 upper=0.2 effort=55 velocity=29
- joint r3_joint_1_to_2: limit lower=-1.2 upper=1.2 effort=10 velocity=200 -> lower=-1.2 upper=1.2 effort=55 velocity=29
- joint r3_joint_2_to_3: limit lower=-0.75 upper=0.2 effort=10 velocity=90 -> lower=-0.75 upper=0.2 effort=55 velocity=29
- joint r3_joint_3_to_4_FOOT: limit lower=-0.5 upper=0.2 effort=10 velocity=70 -> lower=-0.5 upper=0.2 effort=55 velocity=29

File: resources/robots/v0/urdf/v0.urdf.xacro (robot description, xacro)
@@ -45,5 +45,5 @@
 			<origin xyz="0 0 0.25" rpy="0 0 0" />
 			<axis xyz="0.0 0.0 1.0" />
-			<limit effort="10" lower="-1.2" upper="1.2" velocity="200"/>
+			<limit effort="55" lower="-1.2" upper="1.2" velocity="29"/>
 		</joint>
 		<link name="${name}_segment_3_THIGH">
@@ -58,8 +58,8 @@
 			<axis xyz="1.0 0.0 0.0" />
 			<xacro:if value="${reflect == -1}">
-				<limit effort="10" lower="-0.75" upper="0.2" velocity="90"/>
+				<limit effort="55" lower="-0.75" upper="0.2" velocity="29"/>
 			</xacro:if>
 			<xacro:unless value="${reflect == -1}">
-				<limit effort="10" lower="-0.2" upper="0.75" velocity="90"/>
+				<limit effort="55" lower="-0.2" upper="0.75" velocity="29"/>
 			</xacro:unless>
 		</joint>
@@ -75,8 +75,8 @@
 			<axis xyz="1.0 0.0 0.0" />
 			<xacro:if value="${reflect == -1}">
-				<limit effort="10" lower="-0.5" upper="0.2" velocity="70"/>
+				<limit effort="55" lower="-0.5" upper="0.2" velocity="29"/>
 			</xacro:if>
 			<xacro:unless value="${reflect == -1}">
-				<limit effort="10" lower="-0.2" upper="0.5" velocity="70"/>
+				<limit effort="55" lower="-0.2" upper="0.5" velocity="29"/>
 			</xacro:unless>
 		</joint>

Commit message: Make robot significantly heavier

File: resources/robots/v0/urdf/v0.urdf (robot description, URDF)
Before this commit: robot v0, 17 links, 16 joints
Links:
- link body: mass 6.240000000000001 -> 99.84000000000002
- link l1_segment_1: mass 0.32000000000000006 -> 5.120000000000001
- link l1_segment_2_HIP: mass 0.96 -> 15.36
- link l1_segment_3_THIGH: mass 1.12 -> 17.92
- link l1_segment_4_FOOT: mass 0.6400000000000001 -> 10.240000000000002
- link l3_segment_1: mass 0.32000000000000006 -> 5.120000000000001
- link l3_segment_2_HIP: mass 0.96 -> 15.36
- link l3_segment_3_THIGH: mass 1.12 -> 17.92
- link l3_segment_4_FOOT: mass 0.6400000000000001 -> 10.240000000000002
- link r1_segment_1: mass 0.32000000000000006 -> 5.120000000000001
- link r1_segment_2_HIP: mass 0.96 -> 15.36
- link r1_segment_3_THIGH: mass 1.12 -> 17.92
- link r1_segment_4_FOOT: mass 0.6400000000000001 -> 10.240000000000002
- link r3_segment_1: mass 0.32000000000000006 -> 5.120000000000001
- link r3_segment_2_HIP: mass 0.96 -> 15.36
- link r3_segment_3_THIGH: mass 1.12 -> 17.92
- link r3_segment_4_FOOT: mass 0.6400000000000001 -> 10.240000000000002
Joints:
- joint l1_joint_1_to_2: limit lower=-1.2 upper=1.2 effort=55 velocity=29 -> lower=-1.2 upper=1.2 effort=2048 velocity=29
- joint l1_joint_2_to_3: limit lower=-0.2 upper=0.75 effort=55 velocity=29 -> lower=-0.2 upper=0.75 effort=2048 velocity=29
- joint l1_joint_3_to_4_FOOT: limit lower=-0.2 upper=0.5 effort=55 velocity=29 -> lower=-0.2 upper=0.5 effort=2048 velocity=29
- joint l3_joint_1_to_2: limit lower=-1.2 upper=1.2 effort=55 velocity=29 -> lower=-1.2 upper=1.2 effort=2048 velocity=29
- joint l3_joint_2_to_3: limit lower=-0.2 upper=0.75 effort=55 velocity=29 -> lower=-0.2 upper=0.75 effort=2048 velocity=29
- joint l3_joint_3_to_4_FOOT: limit lower=-0.2 upper=0.5 effort=55 velocity=29 -> lower=-0.2 upper=0.5 effort=2048 velocity=29
- joint r1_joint_1_to_2: limit lower=-1.2 upper=1.2 effort=55 velocity=29 -> lower=-1.2 upper=1.2 effort=2048 velocity=29
- joint r1_joint_2_to_3: limit lower=-0.75 upper=0.2 effort=55 velocity=29 -> lower=-0.75 upper=0.2 effort=2048 velocity=29
- joint r1_joint_3_to_4_FOOT: limit lower=-0.5 upper=0.2 effort=55 velocity=29 -> lower=-0.5 upper=0.2 effort=2048 velocity=29
- joint r3_joint_1_to_2: limit lower=-1.2 upper=1.2 effort=55 velocity=29 -> lower=-1.2 upper=1.2 effort=2048 velocity=29
- joint r3_joint_2_to_3: limit lower=-0.75 upper=0.2 effort=55 velocity=29 -> lower=-0.75 upper=0.2 effort=2048 velocity=29
- joint r3_joint_3_to_4_FOOT: limit lower=-0.5 upper=0.2 effort=55 velocity=29 -> lower=-0.5 upper=0.2 effort=2048 velocity=29

File: resources/robots/v0/urdf/v0.urdf.xacro (robot description, xacro)
@@ -16,5 +16,5 @@
         </collision>
 		<inertial>
-			<xacro:property name="weight" value="${sizeX * sizeY * sizeZ * 160}"/>
+			<xacro:property name="weight" value="${sizeX * sizeY * sizeZ * 160 * 16}"/>
 			<mass value="${weight}"/>
 			<inertia
@@ -46,5 +46,5 @@
 			<origin xyz="0 0 0.25" rpy="0 0 0" />
 			<axis xyz="0.0 0.0 1.0" />
-			<limit effort="55" lower="-1.2" upper="1.2" velocity="29"/>
+			<limit effort="2048" lower="-1.2" upper="1.2" velocity="29"/>
 		</joint>
 		<link name="${name}_segment_3_THIGH">
@@ -59,8 +59,8 @@
 			<axis xyz="1.0 0.0 0.0" />
 			<xacro:if value="${reflect == -1}">
-				<limit effort="55" lower="-0.75" upper="0.2" velocity="29"/>
+				<limit effort="2048" lower="-0.75" upper="0.2" velocity="29"/>
 			</xacro:if>
 			<xacro:unless value="${reflect == -1}">
-				<limit effort="55" lower="-0.2" upper="0.75" velocity="29"/>
+				<limit effort="2048" lower="-0.2" upper="0.75" velocity="29"/>
 			</xacro:unless>
 		</joint>
@@ -76,8 +76,8 @@
 			<axis xyz="1.0 0.0 0.0" />
 			<xacro:if value="${reflect == -1}">
-				<limit effort="55" lower="-0.5" upper="0.2" velocity="29"/>
+				<limit effort="2048" lower="-0.5" upper="0.2" velocity="29"/>
 			</xacro:if>
 			<xacro:unless value="${reflect == -1}">
-				<limit effort="55" lower="-0.2" upper="0.5" velocity="29"/>
+				<limit effort="2048" lower="-0.2" upper="0.5" velocity="29"/>
 			</xacro:unless>
 		</joint>

Commit message: Generalize code for six and four legged robots

File: resources/robots/v0/urdf/v0.urdf (robot description, URDF)
Before this commit: robot v0, 17 links, 16 joints
Joints:
- joint l1_joint_1_to_2: limit lower=-1.2 upper=1.2 effort=2048 velocity=29 -> lower=-1.2 upper=1.2 effort=2048 velocity=15
- joint l1_joint_2_to_3: limit lower=-0.2 upper=0.75 effort=2048 velocity=29 -> lower=-0.2 upper=0.75 effort=2048 velocity=15
- joint l1_joint_3_to_4_FOOT: limit lower=-0.2 upper=0.5 effort=2048 velocity=29 -> lower=-0.2 upper=0.5 effort=2048 velocity=9
- joint l3_joint_1_to_2: limit lower=-1.2 upper=1.2 effort=2048 velocity=29 -> lower=-1.2 upper=1.2 effort=2048 velocity=15
- joint l3_joint_2_to_3: limit lower=-0.2 upper=0.75 effort=2048 velocity=29 -> lower=-0.2 upper=0.75 effort=2048 velocity=15
- joint l3_joint_3_to_4_FOOT: limit lower=-0.2 upper=0.5 effort=2048 velocity=29 -> lower=-0.2 upper=0.5 effort=2048 velocity=9
- joint r1_joint_1_to_2: limit lower=-1.2 upper=1.2 effort=2048 velocity=29 -> lower=-1.2 upper=1.2 effort=2048 velocity=15
- joint r1_joint_2_to_3: limit lower=-0.75 upper=0.2 effort=2048 velocity=29 -> lower=-0.75 upper=0.2 effort=2048 velocity=15
- joint r1_joint_3_to_4_FOOT: limit lower=-0.5 upper=0.2 effort=2048 velocity=29 -> lower=-0.5 upper=0.2 effort=2048 velocity=9
- joint r3_joint_1_to_2: limit lower=-1.2 upper=1.2 effort=2048 velocity=29 -> lower=-1.2 upper=1.2 effort=2048 velocity=15
- joint r3_joint_2_to_3: limit lower=-0.75 upper=0.2 effort=2048 velocity=29 -> lower=-0.75 upper=0.2 effort=2048 velocity=15
- joint r3_joint_3_to_4_FOOT: limit lower=-0.5 upper=0.2 effort=2048 velocity=29 -> lower=-0.5 upper=0.2 effort=2048 velocity=9

File: resources/robots/v0/urdf/v0.urdf.xacro (robot description, xacro)
@@ -46,5 +46,5 @@
 			<origin xyz="0 0 0.25" rpy="0 0 0" />
 			<axis xyz="0.0 0.0 1.0" />
-			<limit effort="2048" lower="-1.2" upper="1.2" velocity="29"/>
+			<limit effort="2048" lower="-1.2" upper="1.2" velocity="20"/>
 		</joint>
 		<link name="${name}_segment_3_THIGH">
@@ -59,8 +59,8 @@
 			<axis xyz="1.0 0.0 0.0" />
 			<xacro:if value="${reflect == -1}">
-				<limit effort="2048" lower="-0.75" upper="0.2" velocity="29"/>
+				<limit effort="2048" lower="-0.75" upper="0.2" velocity="20"/>
 			</xacro:if>
 			<xacro:unless value="${reflect == -1}">
-				<limit effort="2048" lower="-0.2" upper="0.75" velocity="29"/>
+				<limit effort="2048" lower="-0.2" upper="0.75" velocity="20"/>
 			</xacro:unless>
 		</joint>
@@ -76,8 +76,8 @@
 			<axis xyz="1.0 0.0 0.0" />
 			<xacro:if value="${reflect == -1}">
-				<limit effort="2048" lower="-0.5" upper="0.2" velocity="29"/>
+				<limit effort="2048" lower="-0.5" upper="0.2" velocity="20"/>
 			</xacro:if>
 			<xacro:unless value="${reflect == -1}">
-				<limit effort="2048" lower="-0.2" upper="0.5" velocity="29"/>
+				<limit effort="2048" lower="-0.2" upper="0.5" velocity="20"/>
 			</xacro:unless>
 		</joint>

File: resources/robots/v0six/urdf/v0.urdf (robot description, URDF)
Before this commit: robot v0, 25 links, 24 joints
Links:
- link body: mass 6.240000000000001 -> 99.84000000000002
- link l1_segment_1: mass 0.32000000000000006 -> 5.120000000000001
- link l1_segment_2_HIP: mass 0.96 -> 15.36
- link l1_segment_3_THIGH: mass 1.12 -> 17.92
- link l1_segment_4_FOOT: mass 0.6400000000000001 -> 10.240000000000002
- link l2_segment_1: mass 0.32000000000000006 -> 5.120000000000001
- link l2_segment_2_HIP: mass 0.96 -> 15.36
- link l2_segment_3_THIGH: mass 1.12 -> 17.92
- link l2_segment_4_FOOT: mass 0.6400000000000001 -> 10.240000000000002
- link l3_segment_1: mass 0.32000000000000006 -> 5.120000000000001
- link l3_segment_2_HIP: mass 0.96 -> 15.36
- link l3_segment_3_THIGH: mass 1.12 -> 17.92
- link l3_segment_4_FOOT: mass 0.6400000000000001 -> 10.240000000000002
- link r1_segment_1: mass 0.32000000000000006 -> 5.120000000000001
- link r1_segment_2_HIP: mass 0.96 -> 15.36
- link r1_segment_3_THIGH: mass 1.12 -> 17.92
- link r1_segment_4_FOOT: mass 0.6400000000000001 -> 10.240000000000002
- link r2_segment_1: mass 0.32000000000000006 -> 5.120000000000001
- link r2_segment_2_HIP: mass 0.96 -> 15.36
- link r2_segment_3_THIGH: mass 1.12 -> 17.92
- link r2_segment_4_FOOT: mass 0.6400000000000001 -> 10.240000000000002
- link r3_segment_1: mass 0.32000000000000006 -> 5.120000000000001
- link r3_segment_2_HIP: mass 0.96 -> 15.36
- link r3_segment_3_THIGH: mass 1.12 -> 17.92
- link r3_segment_4_FOOT: mass 0.6400000000000001 -> 10.240000000000002
Joints:
- joint l1_joint_1_to_2: limit lower=-1.2 upper=1.2 effort=55 velocity=29 -> lower=-1.2 upper=1.2 effort=2048 velocity=20
- joint l1_joint_2_to_3: limit lower=-0.2 upper=0.75 effort=55 velocity=29 -> lower=-0.2 upper=0.75 effort=2048 velocity=20
- joint l1_joint_3_to_4_FOOT: limit lower=-0.2 upper=0.5 effort=55 velocity=29 -> lower=-0.2 upper=0.5 effort=2048 velocity=20
- joint l2_joint_1_to_2: limit lower=-1.2 upper=1.2 effort=55 velocity=29 -> lower=-1.2 upper=1.2 effort=2048 velocity=20
- joint l2_joint_2_to_3: limit lower=-0.2 upper=0.75 effort=55 velocity=29 -> lower=-0.2 upper=0.75 effort=2048 velocity=20
- joint l2_joint_3_to_4_FOOT: limit lower=-0.2 upper=0.5 effort=55 velocity=29 -> lower=-0.2 upper=0.5 effort=2048 velocity=20
- joint l3_joint_1_to_2: limit lower=-1.2 upper=1.2 effort=55 velocity=29 -> lower=-1.2 upper=1.2 effort=2048 velocity=20
- joint l3_joint_2_to_3: limit lower=-0.2 upper=0.75 effort=55 velocity=29 -> lower=-0.2 upper=0.75 effort=2048 velocity=20
- joint l3_joint_3_to_4_FOOT: limit lower=-0.2 upper=0.5 effort=55 velocity=29 -> lower=-0.2 upper=0.5 effort=2048 velocity=20
- joint r1_joint_1_to_2: limit lower=-1.2 upper=1.2 effort=55 velocity=29 -> lower=-1.2 upper=1.2 effort=2048 velocity=20
- joint r1_joint_2_to_3: limit lower=-0.75 upper=0.2 effort=55 velocity=29 -> lower=-0.75 upper=0.2 effort=2048 velocity=20
- joint r1_joint_3_to_4_FOOT: limit lower=-0.5 upper=0.2 effort=55 velocity=29 -> lower=-0.5 upper=0.2 effort=2048 velocity=20
- joint r2_joint_1_to_2: limit lower=-1.2 upper=1.2 effort=55 velocity=29 -> lower=-1.2 upper=1.2 effort=2048 velocity=20
- joint r2_joint_2_to_3: limit lower=-0.75 upper=0.2 effort=55 velocity=29 -> lower=-0.75 upper=0.2 effort=2048 velocity=20
- joint r2_joint_3_to_4_FOOT: limit lower=-0.5 upper=0.2 effort=55 velocity=29 -> lower=-0.5 upper=0.2 effort=2048 velocity=20
- joint r3_joint_1_to_2: limit lower=-1.2 upper=1.2 effort=55 velocity=29 -> lower=-1.2 upper=1.2 effort=2048 velocity=20
- joint r3_joint_2_to_3: limit lower=-0.75 upper=0.2 effort=55 velocity=29 -> lower=-0.75 upper=0.2 effort=2048 velocity=20
- joint r3_joint_3_to_4_FOOT: limit lower=-0.5 upper=0.2 effort=55 velocity=29 -> lower=-0.5 upper=0.2 effort=2048 velocity=20

File: resources/robots/v0six/urdf/v0.urdf.xacro (robot description, xacro)
@@ -16,5 +16,5 @@
         </collision>
 		<inertial>
-			<xacro:property name="weight" value="${sizeX * sizeY * sizeZ * 160}"/>
+			<xacro:property name="weight" value="${sizeX * sizeY * sizeZ * 160 * 16}"/>
 			<mass value="${weight}"/>
 			<inertia
@@ -46,5 +46,5 @@
 			<origin xyz="0 0 0.25" rpy="0 0 0" />
 			<axis xyz="0.0 0.0 1.0" />
-			<limit effort="55" lower="-1.2" upper="1.2" velocity="29"/>
+			<limit effort="2048" lower="-1.2" upper="1.2" velocity="20"/>
 		</joint>
 		<link name="${name}_segment_3_THIGH">
@@ -59,8 +59,8 @@
 			<axis xyz="1.0 0.0 0.0" />
 			<xacro:if value="${reflect == -1}">
-				<limit effort="55" lower="-0.75" upper="0.2" velocity="29"/>
+				<limit effort="2048" lower="-0.75" upper="0.2" velocity="20"/>
 			</xacro:if>
 			<xacro:unless value="${reflect == -1}">
-				<limit effort="55" lower="-0.2" upper="0.75" velocity="29"/>
+				<limit effort="2048" lower="-0.2" upper="0.75" velocity="20"/>
 			</xacro:unless>
 		</joint>
@@ -76,8 +76,8 @@
 			<axis xyz="1.0 0.0 0.0" />
 			<xacro:if value="${reflect == -1}">
-				<limit effort="55" lower="-0.5" upper="0.2" velocity="29"/>
+				<limit effort="2048" lower="-0.5" upper="0.2" velocity="20"/>
 			</xacro:if>
 			<xacro:unless value="${reflect == -1}">
-				<limit effort="55" lower="-0.2" upper="0.5" velocity="29"/>
+				<limit effort="2048" lower="-0.2" upper="0.5" velocity="20"/>
 			</xacro:unless>
 		</joint>
