Commit message: Parametrize v0 xacro file

File: resources/robots/v0six/urdf/v0.urdf (robot description, URDF)
Before this commit: robot v0, 25 links, 24 joints
Joints:
- joint l1_joint_1_to_2: limit lower=-1.2 upper=1.2 effort=2048 velocity=20 -> lower=-1.2 upper=1.2 effort=2048 velocity=3.2
- joint l1_joint_2_to_3: limit lower=-0.2 upper=0.75 effort=2048 velocity=20 -> lower=-0.2 upper=0.75 effort=2048 velocity=3.2
- joint l1_joint_3_to_4_FOOT: limit lower=-0.2 upper=0.5 effort=2048 velocity=20 -> lower=-0.2 upper=0.5 effort=2048 velocity=3.2
- joint l2_joint_1_to_2: limit lower=-1.2 upper=1.2 effort=2048 velocity=20 -> lower=-1.2 upper=1.2 effort=2048 velocity=3.2
- joint l2_joint_2_to_3: limit lower=-0.2 upper=0.75 effort=2048 velocity=20 -> lower=-0.2 upper=0.75 effort=2048 velocity=3.2
- joint l2_joint_3_to_4_FOOT: limit lower=-0.2 upper=0.5 effort=2048 velocity=20 -> lower=-0.2 upper=0.5 effort=2048 velocity=3.2
- joint l3_joint_1_to_2: limit lower=-1.2 upper=1.2 effort=2048 velocity=20 -> lower=-1.2 upper=1.2 effort=2048 velocity=3.2
- joint l3_joint_2_to_3: limit lower=-0.2 upper=0.75 effort=2048 velocity=20 -> lower=-0.2 upper=0.75 effort=2048 velocity=3.2
- joint l3_joint_3_to_4_FOOT: limit lower=-0.2 upper=0.5 effort=2048 velocity=20 -> lower=-0.2 upper=0.5 effort=2048 velocity=3.2
- joint r1_joint_1_to_2: limit lower=-1.2 upper=1.2 effort=2048 velocity=20 -> lower=-1.2 upper=1.2 effort=2048 velocity=3.2
- joint r1_joint_2_to_3: limit lower=-0.75 upper=0.2 effort=2048 velocity=20 -> lower=-0.75 upper=0.2 effort=2048 velocity=3.2
- joint r1_joint_3_to_4_FOOT: limit lower=-0.5 upper=0.2 effort=2048 velocity=20 -> lower=-0.5 upper=0.2 effort=2048 velocity=3.2
- joint r2_joint_1_to_2: limit lower=-1.2 upper=1.2 effort=2048 velocity=20 -> lower=-1.2 upper=1.2 effort=2048 velocity=3.2
- joint r2_joint_2_to_3: limit lower=-0.75 upper=0.2 effort=2048 velocity=20 -> lower=-0.75 upper=0.2 effort=2048 velocity=3.2
- joint r2_joint_3_to_4_FOOT: limit lower=-0.5 upper=0.2 effort=2048 velocity=20 -> lower=-0.5 upper=0.2 effort=2048 velocity=3.2
- joint r3_joint_1_to_2: limit lower=-1.2 upper=1.2 effort=2048 velocity=20 -> lower=-1.2 upper=1.2 effort=2048 velocity=3.2
- joint r3_joint_2_to_3: limit lower=-0.75 upper=0.2 effort=2048 velocity=20 -> lower=-0.75 upper=0.2 effort=2048 velocity=3.2
- joint r3_joint_3_to_4_FOOT: limit lower=-0.5 upper=0.2 effort=2048 velocity=20 -> lower=-0.5 upper=0.2 effort=2048 velocity=3.2

File: resources/robots/v0six/urdf/v0.urdf.xacro (robot description, xacro)
@@ -1,5 +1,8 @@
 <?xml version="1.0"?>
 <robot xmlns:xacro="http://www.ros.org/wiki/xacro" name="v0">
-	<xacro:macro name="box" params="sizeX sizeY sizeZ color *origin">
+	<xacro:property name="VELOCITY" value="3.2"/>
+	<xacro:property name="FRICTION" value="0"/>
+	<xacro:property name="EFFORT" value="2048"/>
+	<xacro:macro name="box" params="sizeX sizeY sizeZ color weight_multiplier:=160 *origin">
 		<visual>
 			<geometry>
@@ -16,5 +19,5 @@
         </collision>
 		<inertial>
-			<xacro:property name="weight" value="${sizeX * sizeY * sizeZ * 160 * 16}"/>
+			<xacro:property name="weight" value="${sizeX * sizeY * sizeZ * 16 * weight_multiplier}"/>
 			<mass value="${weight}"/>
 			<inertia
@@ -35,4 +38,5 @@
 			<child link="${name}_segment_1" />
 			<xacro:insert_block name="origin" />
+			<dynamics damping="0.0" friction="${FRICTION}"/>
 		</joint>
 		<link name="${name}_segment_2_HIP">
@@ -46,5 +50,6 @@
 			<origin xyz="0 0 0.25" rpy="0 0 0" />
 			<axis xyz="0.0 0.0 1.0" />
-			<limit effort="2048" lower="-1.2" upper="1.2" velocity="20"/>
+			<limit effort="${EFFORT}" lower="-1.2" upper="1.2" velocity="${VELOCITY}"/>
+			<dynamics damping="0.0" friction="${FRICTION}"/>
 		</joint>
 		<link name="${name}_segment_3_THIGH">
@@ -59,9 +64,10 @@
 			<axis xyz="1.0 0.0 0.0" />
 			<xacro:if value="${reflect == -1}">
-				<limit effort="2048" lower="-0.75" upper="0.2" velocity="20"/>
+				<limit effort="${EFFORT}" lower="-0.75" upper="0.2" velocity="${VELOCITY}"/>
 			</xacro:if>
 			<xacro:unless value="${reflect == -1}">
-				<limit effort="2048" lower="-0.2" upper="0.75" velocity="20"/>
+				<limit effort="${EFFORT}" lower="-0.2" upper="0.75" velocity="${VELOCITY}"/>
 			</xacro:unless>
+			<dynamics damping="0.0" friction="${FRICTION}"/>
 		</joint>
 		<link name="${name}_segment_4_FOOT">
@@ -76,9 +82,10 @@
 			<axis xyz="1.0 0.0 0.0" />
 			<xacro:if value="${reflect == -1}">
-				<limit effort="2048" lower="-0.5" upper="0.2" velocity="20"/>
+				<limit effort="${EFFORT}" lower="-0.5" upper="0.2" velocity="${VELOCITY}"/>
 			</xacro:if>
 			<xacro:unless value="${reflect == -1}">
-				<limit effort="2048" lower="-0.2" upper="0.5" velocity="20"/>
+				<limit effort="${EFFORT}" lower="-0.2" upper="0.5" velocity="${VELOCITY}"/>
 			</xacro:unless>
+			<dynamics damping="0.0" friction="${FRICTION}"/>
 		</joint>
 	</xacro:macro>
